Commit message: feat(description): switch ros2_control to effort interface for CHAMP
CHAMP's quadruped_controller drives joints via effort. The gazebo plugin
now reads its yaml from dog_robot_config so the controller list / gains
travel with the config package rather than being hardcoded in the URDF.

Co-Authored-By: Claude Opus 4.7 (1M context) <noreply@anthropic.com>

File: dog_robot_ws/src/dog_robot_description/urdf/gazebo.xacro (robot description, xacro)
@@ -5,9 +5,10 @@
       <mu1>1.0</mu1>
       <mu2>1.0</mu2>
-      <kp>1000000.0</kp>
-      <kd>100.0</kd>
+      <kp>1000.0</kp>
+      <kd>1.0</kd>
       <minDepth>0.001</minDepth>
       <maxVel>0.1</maxVel>
       <material>Gazebo/DarkGrey</material>
+      <self_collide>false</self_collide>
     </gazebo>
   </xacro:macro>
@@ -16,18 +17,31 @@
   <xacro:foot_friction prefix="BL"/>
   <xacro:foot_friction prefix="BR"/>
+  <xacro:macro name="no_self_collide" params="link">
+    <gazebo reference="${link}">
+      <self_collide>false</self_collide>
+    </gazebo>
+  </xacro:macro>
+  <!-- Hip meshes overlap base_link bbox; thigh/shank chain may also
+       overlap adjacent links. Disable self-collision on every leg
+       link so ODE doesn't apply huge separation impulses at spawn. -->
+  <xacro:no_self_collide link="FL_hip_link"/>
+  <xacro:no_self_collide link="FL_thigh_link"/>
+  <xacro:no_self_collide link="FL_shank_link"/>
+  <xacro:no_self_collide link="FR_hip_link"/>
+  <xacro:no_self_collide link="FR_thigh_link"/>
+  <xacro:no_self_collide link="FR_shank_link"/>
+  <xacro:no_self_collide link="BL_hip_link"/>
+  <xacro:no_self_collide link="BL_thigh_link"/>
+  <xacro:no_self_collide link="BL_shank_link"/>
+  <xacro:no_self_collide link="BR_hip_link"/>
+  <xacro:no_self_collide link="BR_thigh_link"/>
+  <xacro:no_self_collide link="BR_shank_link"/>
   <gazebo reference="base_link">
     <material>Gazebo/Grey</material>
     <self_collide>false</self_collide>
   </gazebo>
-  <!--
-    The gazebo_ros2_control plugin hangs at startup when the <parameters>
-    tag contains a $(find ...) substitution. Pass the absolute path in
-    via a xacro arg from the launch file so what reaches Gazebo is a
-    plain string.
-  -->
-  <xacro:arg name="controllers_yaml_path" default=""/>
   <gazebo>
     <plugin filename="libgazebo_ros2_control.so" name="gazebo_ros2_control">
-      <parameters>$(arg controllers_yaml_path)</parameters>
+      <parameters>$(find dog_robot_config)/config/ros_control/ros_control.yaml</parameters>
     </plugin>
   </gazebo>

File: dog_robot_ws/src/dog_robot_description/urdf/ros2_control.xacro (robot description, xacro)
@@ -3,7 +3,7 @@
   <xacro:macro name="joint_iface" params="name lower upper">
     <joint name="${name}">
-      <command_interface name="position">
-        <param name="min">${lower}</param>
-        <param name="max">${upper}</param>
+      <command_interface name="effort">
+        <param name="min">-2.0</param>
+        <param name="max">2.0</param>
       </command_interface>
       <state_interface name="position"/>

Commit message: tune(stand): fix Gazebo stand verification — position interface + corrected height
Five root causes resolved:

1. gazebo.xacro hardcoded CHAMP ros_control.yaml as the gazebo_ros2_control
   plugin parameters, so stand.launch.py could never load its own controller
   types. Added xacro:arg controllers_yaml_path (default = CHAMP yaml so
   dog_robot_config launches are unaffected) and plumb it through <parameters>.

2. default_height 0.18 m exceeded leg reach: FK analysis showed the IK
   solver needed dist=0.1896 m but max reach = L_th+L_sh = 0.1877 m.
   Height reduced to 0.15 m (a_t = 0.1596 m, well within reach).

3. JTC effort interface with PID caused ODE physics divergence (joint
   velocities 50–60 rad/s). Switched JTC to position command interface
   + open_loop_control: true; gazebo_ros2_control handles position
   tracking natively and stably. Removed PID gains block.

4. ros2_control.xacro now also declares position command interface
   (alongside effort, which CHAMP still uses) so both paths co-exist.

5. Joint damping raised 0.05→0.50, effort limit 5→10 Nm to support
   the position controller and prevent post-contact bounce.

Verified: all 12 joints converge to hip=0, thigh=-0.4145, knee=+1.1495
within 2 s ramp; steady-state max velocity <0.53 rad/s; body z ≈ 0.168 m;
roll ≈ 0, pitch ≈ 0 (symmetric stance).

Co-Authored-By: Claude Sonnet 4.6 <noreply@anthropic.com>

File: dog_robot_ws/src/dog_robot_description/urdf/gazebo.xacro (robot description, xacro)
@@ -41,7 +41,12 @@
     <self_collide>false</self_collide>
   </gazebo>
+  <!-- controllers_yaml_path can be overridden at xacro time; falls back to
+       the CHAMP ros_control.yaml so the dog_robot_config/launch/gazebo.launch.py
+       path continues to work unchanged. -->
+  <xacro:arg name="controllers_yaml_path"
+             default="$(find dog_robot_config)/config/ros_control/ros_control.yaml"/>
   <gazebo>
     <plugin filename="libgazebo_ros2_control.so" name="gazebo_ros2_control">
-      <parameters>$(find dog_robot_config)/config/ros_control/ros_control.yaml</parameters>
+      <parameters>$(arg controllers_yaml_path)</parameters>
     </plugin>
   </gazebo>

File: dog_robot_ws/src/dog_robot_description/urdf/leg.xacro (robot description, xacro)
@@ -30,6 +30,6 @@
       <origin xyz="${base_to_hip_xyz}" rpy="${base_to_hip_rpy}"/>
       <axis xyz="0 0 1"/>
-      <limit lower="-0.785" upper="0.785" effort="5.0" velocity="8.0"/>
-      <dynamics damping="0.05" friction="0.0"/>
+      <limit lower="-0.785" upper="0.785" effort="10.0" velocity="8.0"/>
+      <dynamics damping="0.5" friction="0.0"/>
     </joint>
     <link name="${prefix}_thigh_link">
@@ -54,6 +54,6 @@
       <origin xyz="${L_hh} 0 0" rpy="-1.5707963 0 0"/>
       <axis xyz="0 0 1"/>
-      <limit lower="-1.571" upper="1.571" effort="5.0" velocity="8.0"/>
-      <dynamics damping="0.05" friction="0.0"/>
+      <limit lower="-1.571" upper="1.571" effort="10.0" velocity="8.0"/>
+      <dynamics damping="0.5" friction="0.0"/>
     </joint>
     <link name="${prefix}_shank_link">
@@ -78,6 +78,6 @@
       <origin xyz="${L_th} 0 0" rpy="0 0 0"/>
       <axis xyz="0 0 1"/>
-      <limit lower="0.0" upper="2.617" effort="5.0" velocity="8.0"/>
-      <dynamics damping="0.05" friction="0.0"/>
+      <limit lower="0.0" upper="2.617" effort="10.0" velocity="8.0"/>
+      <dynamics damping="0.5" friction="0.0"/>
     </joint>
     <link name="${prefix}_foot_link">

File: dog_robot_ws/src/dog_robot_description/urdf/ros2_control.xacro (robot description, xacro)
@@ -3,4 +3,8 @@
   <xacro:macro name="joint_iface" params="name lower upper">
     <joint name="${name}">
+      <command_interface name="position">
+        <param name="min">${lower}</param>
+        <param name="max">${upper}</param>
+      </command_interface>
       <command_interface name="effort"/>
       <state_interface name="position"/>
