Commit message: fix(meshes): use CAD-measured joint positions for re-centering + xacro origins

File: dog_robot_ws/src/dog_robot_description/urdf/dog_robot.urdf.xacro (robot description, xacro)
@@ -24,7 +24,24 @@
     </xacro:inertial_box>
   </link>
-  <xacro:leg prefix="FL" x_offset=" 0.100" y_offset=" 0.040" y_sign=" 1"/>
-  <xacro:leg prefix="FR" x_offset=" 0.100" y_offset="-0.040" y_sign="-1"/>
-  <xacro:leg prefix="BL" x_offset="-0.100" y_offset=" 0.040" y_sign=" 1"/>
-  <xacro:leg prefix="BR" x_offset="-0.100" y_offset="-0.040" y_sign="-1"/>
+  <!-- Joint origins measured from CAD (scripts/compute_joints.py). -->
+  <xacro:leg prefix="FL"
+             hip_xyz="0.10180 0.04342 0.02667"
+             thigh_xyz="-0.02099 0.02033 -0.01287"
+             knee_xyz="-0.03799 0.02250 -0.03872"
+             foot_xyz="0.02489 0.00091 -0.05492"/>
+  <xacro:leg prefix="FR"
+             hip_xyz="0.10180 -0.04362 0.02677"
+             thigh_xyz="-0.02084 -0.02075 -0.01264"
+             knee_xyz="-0.03756 -0.02348 -0.03881"
+             foot_xyz="0.02499 -0.00229 -0.05544"/>
+  <xacro:leg prefix="BL"
+             hip_xyz="-0.10373 0.04342 0.02667"
+             thigh_xyz="-0.01730 0.02029 -0.01459"
+             knee_xyz="-0.03206 0.02242 -0.04137"
+             foot_xyz="0.02987 0.00100 -0.05074"/>
+  <xacro:leg prefix="BR"
+             hip_xyz="-0.10178 -0.04362 0.02677"
+             thigh_xyz="-0.02063 -0.02133 -0.02285"
+             knee_xyz="-0.03221 -0.02338 -0.04135"
+             foot_xyz="0.03222 -0.00166 -0.04264"/>
 </robot>

File: dog_robot_ws/src/dog_robot_description/urdf/leg.xacro (robot description, xacro)
@@ -1,5 +1,7 @@
 <?xml version="1.0"?>
 <robot xmlns:xacro="http://www.ros.org/wiki/xacro" name="dog_robot_leg">
-  <xacro:macro name="leg" params="prefix x_offset y_offset y_sign">
+  <!-- Joint origins are measured from CAD (see scripts/compute_joints.py). -->
+  <xacro:macro name="leg" params="prefix
+                                  hip_xyz thigh_xyz knee_xyz foot_xyz">
     <link name="${prefix}_hip_link">
       <visual>
@@ -23,5 +25,5 @@
       <parent link="base_link"/>
       <child link="${prefix}_hip_link"/>
-      <origin xyz="${x_offset} ${y_offset} 0" rpy="0 0 0"/>
+      <origin xyz="${hip_xyz}" rpy="0 0 0"/>
       <axis xyz="1 0 0"/>
       <limit lower="-0.785" upper="0.785" effort="2.0" velocity="5.0"/>
@@ -49,5 +51,5 @@
       <parent link="${prefix}_hip_link"/>
       <child link="${prefix}_thigh_link"/>
-      <origin xyz="0 ${y_sign * 0.04895} 0" rpy="0 0 0"/>
+      <origin xyz="${thigh_xyz}" rpy="0 0 0"/>
       <axis xyz="0 1 0"/>
       <limit lower="-1.571" upper="1.571" effort="2.0" velocity="5.0"/>
@@ -75,5 +77,5 @@
       <parent link="${prefix}_thigh_link"/>
       <child link="${prefix}_shank_link"/>
-      <origin xyz="0 0 -0.109202" rpy="0 0 0"/>
+      <origin xyz="${knee_xyz}" rpy="0 0 0"/>
       <axis xyz="0 1 0"/>
       <limit lower="0.0" upper="2.617" effort="2.0" velocity="5.0"/>
@@ -101,5 +103,5 @@
       <parent link="${prefix}_shank_link"/>
       <child link="${prefix}_foot_link"/>
-      <origin xyz="0 0 -0.115" rpy="0 0 0"/>
+      <origin xyz="${foot_xyz}" rpy="0 0 0"/>
     </joint>
   </xacro:macro>

Commit message: fix(description): unfreeze Gazebo physics for full 12-DoF robot
Root cause: Gazebo classic 11.10.2 + ODE froze the entire kinematic
tree (base_link + 12 revolute joints) when each non-foot leg link
had no <collision>. Bodies stayed at world origin with NaN joint
velocities and physics never integrated for the model. Reproduced
with a generic 4-link chain; physics only resumed once every link
exposed a <collision> primitive.

Combined with that, joint damping=1.0 with effort_limit=2.0 in a
4+ link chain put ODE in a numerically unstable regime that kept
the model pinned even after adding collisions. Lowering damping
to 0.05 (CHAMP-style) restored normal dynamics.

Changes:
- leg.xacro: add primitive box <collision> to hip/thigh/shank
  links so every body in the tree has a collision shape.
  Self-collisions are already disabled in gazebo.xacro so legs
  do not prop the body up.
- leg.xacro: drop joint damping from 1.0 to 0.05 and friction
  to 0.0 across all 12 joints.
- dog_robot.urdf.xacro / leg.xacro: switch mesh URIs from
  package:// to file://$(find ...) so gz sdf does not rewrite
  them to model:// (which needs model.config to resolve).
- ros2_control.xacro: drop <param>min/max on the effort
  command_interface to match CHAMP's stock setup.

Verified: forward cmd_vel produces base_link x motion and finite
joint velocities; pose remains at z≈0.016 on the ground.

File: dog_robot_ws/src/dog_robot_description/urdf/dog_robot.urdf.xacro (robot description, xacro)
@@ -10,5 +10,5 @@
       <origin xyz="0 0 0" rpy="0 0 0"/>
       <geometry>
-        <mesh filename="package://dog_robot_description/meshes/visual/base_link.stl"/>
+        <mesh filename="file://$(find dog_robot_description)/meshes/visual/base_link.stl"/>
       </geometry>
       <material name="grey"/>
@@ -17,5 +17,5 @@
       <origin xyz="0 0 0" rpy="0 0 0"/>
       <geometry>
-        <mesh filename="package://dog_robot_description/meshes/collision/base_link.stl"/>
+        <mesh filename="file://$(find dog_robot_description)/meshes/collision/base_link.stl"/>
       </geometry>
     </collision>

File: dog_robot_ws/src/dog_robot_description/urdf/leg.xacro (robot description, xacro)
@@ -8,12 +8,15 @@
         <origin xyz="0 0 0" rpy="0 0 0"/>
         <geometry>
-          <mesh filename="package://dog_robot_description/meshes/visual/${prefix}_hip_link.stl"/>
+          <mesh filename="file://$(find dog_robot_description)/meshes/visual/${prefix}_hip_link.stl"/>
         </geometry>
         <material name="grey"/>
       </visual>
+      <!-- Small box collision keeps ODE physics active on this branch.
+           Self-collisions are disabled in gazebo.xacro so legs don't
+           prop the body up. -->
       <collision>
         <origin xyz="0 0 0" rpy="0 0 0"/>
         <geometry>
-          <mesh filename="package://dog_robot_description/meshes/collision/${prefix}_hip_link.stl"/>
+          <box size="0.03 0.03 0.03"/>
         </geometry>
       </collision>
@@ -28,5 +31,5 @@
       <axis xyz="1 0 0"/>
       <limit lower="-0.785" upper="0.785" effort="2.0" velocity="5.0"/>
-      <dynamics damping="0.01" friction="0.0"/>
+      <dynamics damping="0.05" friction="0.0"/>
     </joint>
     <link name="${prefix}_thigh_link">
@@ -34,12 +37,12 @@
         <origin xyz="0 0 0" rpy="0 0 0"/>
         <geometry>
-          <mesh filename="package://dog_robot_description/meshes/visual/${prefix}_thigh_link.stl"/>
+          <mesh filename="file://$(find dog_robot_description)/meshes/visual/${prefix}_thigh_link.stl"/>
         </geometry>
         <material name="dark_grey"/>
       </visual>
       <collision>
-        <origin xyz="0 0 0" rpy="0 0 0"/>
+        <origin xyz="0 0 -0.05" rpy="0 0 0"/>
         <geometry>
-          <mesh filename="package://dog_robot_description/meshes/collision/${prefix}_thigh_link.stl"/>
+          <box size="0.02 0.02 0.08"/>
         </geometry>
       </collision>
@@ -54,5 +57,5 @@
       <axis xyz="0 1 0"/>
       <limit lower="-1.571" upper="1.571" effort="2.0" velocity="5.0"/>
-      <dynamics damping="0.01" friction="0.0"/>
+      <dynamics damping="0.05" friction="0.0"/>
     </joint>
     <link name="${prefix}_shank_link">
@@ -60,12 +63,12 @@
         <origin xyz="0 0 0" rpy="0 0 0"/>
         <geometry>
-          <mesh filename="package://dog_robot_description/meshes/visual/${prefix}_shank_link.stl"/>
+          <mesh filename="file://$(find dog_robot_description)/meshes/visual/${prefix}_shank_link.stl"/>
         </geometry>
         <material name="grey"/>
       </visual>
       <collision>
-        <origin xyz="0 0 0" rpy="0 0 0"/>
+        <origin xyz="0 0 -0.0575" rpy="0 0 0"/>
         <geometry>
-          <mesh filename="package://dog_robot_description/meshes/collision/${prefix}_shank_link.stl"/>
+          <box size="0.015 0.015 0.10"/>
         </geometry>
       </collision>
@@ -80,5 +83,5 @@
       <axis xyz="0 1 0"/>
       <limit lower="0.0" upper="2.617" effort="2.0" velocity="5.0"/>
-      <dynamics damping="0.01" friction="0.0"/>
+      <dynamics damping="0.05" friction="0.0"/>
     </joint>
     <link name="${prefix}_foot_link">
@@ -86,12 +89,13 @@
         <origin xyz="0 0 0" rpy="0 0 0"/>
         <geometry>
-          <mesh filename="package://dog_robot_description/meshes/visual/${prefix}_foot_link.stl"/>
+          <mesh filename="file://$(find dog_robot_description)/meshes/visual/${prefix}_foot_link.stl"/>
         </geometry>
         <material name="dark_grey"/>
       </visual>
+      <!-- Sphere collision (mesh foot caused ODE contact instability). -->
       <collision>
-        <origin xyz="0 0 0" rpy="0 0 0"/>
+        <origin xyz="0.042 0 -0.029" rpy="0 0 0"/>
         <geometry>
-          <mesh filename="package://dog_robot_description/meshes/collision/${prefix}_foot_link.stl"/>
+          <sphere radius="0.018"/>
         </geometry>
       </collision>

File: dog_robot_ws/src/dog_robot_description/urdf/ros2_control.xacro (robot description, xacro)
@@ -3,8 +3,5 @@
   <xacro:macro name="joint_iface" params="name lower upper">
     <joint name="${name}">
-      <command_interface name="effort">
-        <param name="min">-2.0</param>
-        <param name="max">2.0</param>
-      </command_interface>
+      <command_interface name="effort"/>
       <state_interface name="position"/>
       <state_interface name="velocity"/>

Commit message: fix(urdf): bake visual compensation into STL vertices (B2)
The previous visual_*_xyz / visual_*_rpy compensation in URDF kept
mis-rendering meshes because the compensation math is hard to get
right under repeated frame refactors (we just chased two bugs in it).

Move the compensation into the mesh files themselves once:

  scripts/bake_meshes_to_link_frame.py applies the per-leg visual
  origin (as it stood in dog_robot.urdf.xacro at fd3a8db) directly
  onto each STL's vertex coordinates, writing meshes/visual_dh/.

URDF now references meshes/visual_dh/ for every link and uses
identity <visual><origin/> everywhere. leg.xacro drops the
mesh_*_xyz / mesh_*_rpy macro params entirely; dog_robot.urdf.xacro
drops the per-leg paste-in values.

Joint origins, DH lengths, and kinematics_dh are unchanged -- this
is a visual-only refactor. Future DH refactors that re-orient link
frames just need to re-run the bake script with the new compensation
values; the URDF stays clean.

Also fixes the RViz Tools entry (Orbit was a View class).

File: dog_robot_ws/src/dog_robot_description/urdf/dog_robot.urdf.xacro (robot description, xacro)
@@ -10,5 +10,5 @@
       <origin xyz="0 0 0" rpy="0 0 0"/>
       <geometry>
-        <mesh filename="file://$(find dog_robot_description)/meshes/visual/base_link.stl"/>
+        <mesh filename="file://$(find dog_robot_description)/meshes/visual_dh/base_link.stl"/>
       </geometry>
       <material name="grey"/>
@@ -25,7 +25,9 @@
   </link>
   <!-- Modified DH (Craig) configuration. One symmetric DH table for all 4 legs;
-       per-leg variation lives entirely in the base_to_hip_* and mesh_* params.
-       L_hh/L_th/L_sh computed from CAD by scripts/compute_dh_lengths.py;
-       mesh xyz/rpy computed by scripts/compute_visual_compensation.py. -->
+       per-leg variation lives entirely in the base_to_hip_* params.
+       L_hh/L_th/L_sh computed from CAD by scripts/compute_dh_lengths.py.
+       Visual meshes are pre-baked in meshes/visual_dh/ (see
+       scripts/bake_meshes_to_link_frame.py); URDF visual <origin> is
+       identity for every link. -->
   <xacro:property name="L_hh" value="0.02553"/>
   <xacro:property name="L_th" value="0.11725"/>
@@ -35,8 +37,4 @@
              base_to_hip_rpy="0 1.5707963 0"
              L_hh="${L_hh}" L_th="${L_th}" L_sh="${L_sh}"
-             mesh_hip_xyz="0.0 0.0 0.0" mesh_hip_rpy="0.00000 -1.57080 0.00000"
-             mesh_thigh_xyz="-0.01236 -0.0252 0.02536" mesh_thigh_rpy="1.57080 0.00000 -1.57080"
-             mesh_shank_xyz="-0.06506 0.06367 0.06638" mesh_shank_rpy="1.57080 0.00000 -1.57080"
-             mesh_foot_xyz="-0.09828 0.00708 0.04716" mesh_foot_rpy="1.57080 0.00000 -1.57080"
              foot_sphere_xyz="0 0 0"/>
   <xacro:leg prefix="FR"
@@ -44,8 +42,4 @@
              base_to_hip_rpy="0 1.5707963 3.1415927"
              L_hh="${L_hh}" L_th="${L_th}" L_sh="${L_sh}"
-             mesh_hip_xyz="0.0 0.0 0.0" mesh_hip_rpy="0.00000 1.57080 -3.14159"
-             mesh_thigh_xyz="-0.01303 0.0252 0.0257" mesh_thigh_rpy="-1.57080 0.00000 1.57080"
-             mesh_shank_xyz="-0.06561 -0.06279 0.0684" mesh_shank_rpy="-1.57080 0.00000 1.57080"
-             mesh_foot_xyz="-0.09799 -0.00641 0.05014" mesh_foot_rpy="-1.57080 0.00000 1.57080"
              foot_sphere_xyz="0 0 0"/>
   <xacro:leg prefix="BL"
@@ -53,8 +47,4 @@
              base_to_hip_rpy="0 1.5707963 0"
              L_hh="${L_hh}" L_th="${L_th}" L_sh="${L_sh}"
-             mesh_hip_xyz="0.0 0.0 0.0" mesh_hip_rpy="0.00000 -1.57080 0.00000"
-             mesh_thigh_xyz="-0.01235 0.0252 0.02536" mesh_thigh_rpy="1.57080 0.00000 -1.57080"
-             mesh_shank_xyz="-0.05801 0.10861 0.06618" mesh_shank_rpy="1.57080 0.00000 -1.57080"
-             mesh_foot_xyz="-0.09806 0.04842 0.04712" mesh_foot_rpy="1.57080 0.00000 -1.57080"
              foot_sphere_xyz="0 0 0"/>
   <xacro:leg prefix="BR"
@@ -62,8 +52,4 @@
              base_to_hip_rpy="0 1.5707963 3.1415927"
              L_hh="${L_hh}" L_th="${L_th}" L_sh="${L_sh}"
-             mesh_hip_xyz="0.0 0.0 0.0" mesh_hip_rpy="0.00000 1.57080 -3.14159"
-             mesh_thigh_xyz="-0.01303 -0.0252 0.0257" mesh_thigh_rpy="-1.57080 0.00000 1.57080"
-             mesh_shank_xyz="-0.0593 -0.10819 0.0684" mesh_shank_rpy="-1.57080 0.00000 1.57080"
-             mesh_foot_xyz="-0.09804 -0.04759 0.04998" mesh_foot_rpy="-1.57080 0.00000 1.57080"
              foot_sphere_xyz="0 0 0"/>
 </robot>

File: dog_robot_ws/src/dog_robot_description/urdf/leg.xacro (robot description, xacro)
@@ -4,14 +4,10 @@
                                   base_to_hip_xyz base_to_hip_rpy
                                   L_hh L_th L_sh
-                                  mesh_hip_xyz mesh_hip_rpy
-                                  mesh_thigh_xyz mesh_thigh_rpy
-                                  mesh_shank_xyz mesh_shank_rpy
-                                  mesh_foot_xyz mesh_foot_rpy
                                   foot_sphere_xyz:='0 0 0'">
     <link name="${prefix}_hip_link">
       <visual>
-        <origin xyz="${mesh_hip_xyz}" rpy="${mesh_hip_rpy}"/>
+        <origin xyz="0 0 0" rpy="0 0 0"/>
         <geometry>
-          <mesh filename="package://dog_robot_description/meshes/visual/${prefix}_hip_link.stl"/>
+          <mesh filename="package://dog_robot_description/meshes/visual_dh/${prefix}_hip_link.stl"/>
         </geometry>
         <material name="grey"/>
@@ -35,7 +31,7 @@
     <link name="${prefix}_thigh_link">
       <visual>
-        <origin xyz="${mesh_thigh_xyz}" rpy="${mesh_thigh_rpy}"/>
+        <origin xyz="0 0 0" rpy="0 0 0"/>
         <geometry>
-          <mesh filename="package://dog_robot_description/meshes/visual/${prefix}_thigh_link.stl"/>
+          <mesh filename="package://dog_robot_description/meshes/visual_dh/${prefix}_thigh_link.stl"/>
         </geometry>
         <material name="dark_grey"/>
@@ -59,7 +55,7 @@
     <link name="${prefix}_shank_link">
       <visual>
-        <origin xyz="${mesh_shank_xyz}" rpy="${mesh_shank_rpy}"/>
+        <origin xyz="0 0 0" rpy="0 0 0"/>
         <geometry>
-          <mesh filename="package://dog_robot_description/meshes/visual/${prefix}_shank_link.stl"/>
+          <mesh filename="package://dog_robot_description/meshes/visual_dh/${prefix}_shank_link.stl"/>
         </geometry>
         <material name="grey"/>
@@ -83,7 +79,7 @@
     <link name="${prefix}_foot_link">
       <visual>
-        <origin xyz="${mesh_foot_xyz}" rpy="${mesh_foot_rpy}"/>
+        <origin xyz="0 0 0" rpy="0 0 0"/>
         <geometry>
-          <mesh filename="package://dog_robot_description/meshes/visual/${prefix}_foot_link.stl"/>
+          <mesh filename="package://dog_robot_description/meshes/visual_dh/${prefix}_foot_link.stl"/>
         </geometry>
         <material name="dark_grey"/>
