Commit message: fix(description): rotate leg frames so CHAMP IK matches URDF
CHAMP's IK assumes knee_xyz and foot_xyz lie along -Z in their parent
joint frames. Our CAD-derived URDF had knee_xyz.x = -0.089 and
foot_xyz.x = +0.057, which fed a ~+0.94 rad bias into ik_alpha and
caused thigh_pitch to clamp at the joint limit (2.858 rad).

Rotate the thigh_pitch and knee_pitch joint frames by per-leg Ry
amounts so knee_xyz and foot_xyz land on -Z. Apply compensating Ry
to thigh/shank/foot visual meshes so the rendered geometry stays in
the original CAD pose. Re-express the foot collision sphere xyz in
the new rotated foot_link frame.

Joint state at idle now sits within +-0.5 rad on all 12 joints
(vs. 2.858 rad clamp before), and all four feet are below base_link.

Co-Authored-By: Claude Opus 4.7 (1M context) <noreply@anthropic.com>

File: dog_robot_ws/src/dog_robot_description/urdf/dog_robot.urdf.xacro (robot description, xacro)
@@ -24,24 +24,55 @@
     </xacro:inertial_box>
   </link>
-  <!-- Joint origins measured from CAD (scripts/compute_joints.py). -->
+  <!-- Joint origins measured from CAD (scripts/compute_joints.py).
+       The thigh/knee rpy_y values and compensating mesh rpy_y values
+       rotate the thigh and shank link frames so knee_xyz and foot_xyz
+       lie along -Z. This makes CHAMP's IK trivially produce ~0 for
+       thigh_pitch/knee_pitch when the foot is directly below the hip.
+       foot_sphere_xyz is the original (0.042, 0, -0.029) collision
+       sphere offset re-expressed in the rotated foot_link frame:
+       sphere_new = Ry(-(thigh_rpy + knee_rpy)) * sphere_old. -->
   <xacro:leg prefix="FL"
              hip_xyz="0.07480 0.04000 0.03510"
              thigh_xyz="0.02520 0.02536 -0.01317"
-             knee_xyz="-0.08887 0.04102 -0.06455"
-             foot_xyz="0.05659 -0.01922 -0.03721"/>
+             knee_xyz="0.0 0.04102 -0.10984"
+             foot_xyz="0.0 -0.01922 -0.06773"
+             thigh_rpy="0.94261"
+             knee_rpy="-1.93175"
+             mesh_thigh_rpy="-0.94261"
+             mesh_shank_rpy="0.98914"
+             mesh_foot_rpy="0.98914"
+             foot_sphere_xyz="-0.0011 0 -0.0510"/>
   <xacro:leg prefix="FR"
              hip_xyz="0.07480 -0.04000 0.03510"
              thigh_xyz="0.02520 -0.02570 -0.01250"
-             knee_xyz="-0.08799 -0.04270 -0.06467"
-             foot_xyz="0.05638 0.01826 -0.03805"/>
+             knee_xyz="0.0 -0.04270 -0.10920"
+             foot_xyz="0.0 0.01826 -0.06802"
+             thigh_rpy="0.93698"
+             knee_rpy="-1.91411"
+             mesh_thigh_rpy="-0.93698"
+             mesh_shank_rpy="0.97713"
+             mesh_foot_rpy="0.97713"
+             foot_sphere_xyz="-0.0007 0 -0.0511"/>
   <xacro:leg prefix="BL"
              hip_xyz="-0.07480 0.04000 0.03510"
              thigh_xyz="-0.02520 0.02536 -0.01318"
-             knee_xyz="-0.08341 0.04082 -0.07159"
-             foot_xyz="0.06019 -0.01906 -0.03038"/>
+             knee_xyz="0.0 0.04082 -0.10992"
+             foot_xyz="0.0 -0.01906 -0.06742"
+             thigh_rpy="0.86151"
+             knee_rpy="-1.96488"
+             mesh_thigh_rpy="-0.86151"
+             mesh_shank_rpy="1.10337"
+             mesh_foot_rpy="1.10337"
+             foot_sphere_xyz="-0.0071 0 -0.0505"/>
   <xacro:leg prefix="BR"
              hip_xyz="-0.07480 -0.04000 0.03510"
              thigh_xyz="-0.02520 -0.02570 -0.01250"
-             knee_xyz="-0.08299 -0.04270 -0.07098"
-             foot_xyz="0.06059 0.01842 -0.03169"/>
+             knee_xyz="0.0 -0.04270 -0.10920"
+             foot_xyz="0.0 0.01842 -0.06838"
+             thigh_rpy="0.86324"
+             knee_rpy="-1.95214"
+             mesh_thigh_rpy="-0.86324"
+             mesh_shank_rpy="1.08890"
+             mesh_foot_rpy="1.08890"
+             foot_sphere_xyz="-0.0063 0 -0.0507"/>
 </robot>

File: dog_robot_ws/src/dog_robot_description/urdf/leg.xacro (robot description, xacro)
@@ -1,12 +1,30 @@
 <?xml version="1.0"?>
 <robot xmlns:xacro="http://www.ros.org/wiki/xacro" name="dog_robot_leg">
-  <!-- Joint origins are measured from CAD (see scripts/compute_joints.py). -->
+  <!--
+    Joint origins are measured from CAD (see scripts/compute_joints.py).
+    CHAMP-IK-compatible surgery:
+      - thigh_pitch joint frame is rotated by Ry(thigh_rpy) so the
+        knee_xyz lies along -Z (kills ik_alpha bias term).
+      - knee_pitch joint frame is rotated by Ry(knee_rpy) so the
+        foot_xyz lies along -Z (kills ik_beta bias term).
+      - Visual meshes get compensating Ry rotations so the rendered
+        geometry still matches the original CAD pose.
+      - Collision boxes on thigh/shank are reset to xyz=0 rpy=0; the
+        original z-offset was tuned for the un-rotated frame and is
+        not worth re-deriving (boxes are small and approximately
+        symmetric about link origin).
+      - Foot collision sphere xyz must be passed in already expressed
+        in the rotated foot_link frame.
+  -->
   <xacro:macro name="leg" params="prefix
-                                  hip_xyz thigh_xyz knee_xyz foot_xyz">
+                                  hip_xyz thigh_xyz knee_xyz foot_xyz
+                                  thigh_rpy:=0 knee_rpy:=0
+                                  mesh_thigh_rpy:=0 mesh_shank_rpy:=0 mesh_foot_rpy:=0
+                                  foot_sphere_xyz:='0.042 0 -0.029'">
     <link name="${prefix}_hip_link">
       <visual>
         <origin xyz="0 0 0" rpy="0 0 0"/>
         <geometry>
-          <mesh filename="file://$(find dog_robot_description)/meshes/visual/${prefix}_hip_link.stl"/>
+          <mesh filename="package://dog_robot_description/meshes/visual/${prefix}_hip_link.stl"/>
         </geometry>
         <material name="grey"/>
@@ -35,12 +53,12 @@
     <link name="${prefix}_thigh_link">
       <visual>
-        <origin xyz="0 0 0" rpy="0 0 0"/>
+        <origin xyz="0 0 0" rpy="0 ${mesh_thigh_rpy} 0"/>
         <geometry>
-          <mesh filename="file://$(find dog_robot_description)/meshes/visual/${prefix}_thigh_link.stl"/>
+          <mesh filename="package://dog_robot_description/meshes/visual/${prefix}_thigh_link.stl"/>
         </geometry>
         <material name="dark_grey"/>
       </visual>
       <collision>
-        <origin xyz="0 0 -0.05" rpy="0 0 0"/>
+        <origin xyz="0 0 0" rpy="0 0 0"/>
         <geometry>
           <box size="0.02 0.02 0.08"/>
@@ -48,5 +66,5 @@
       </collision>
       <xacro:inertial_box mass="0.10" x="0.03" y="0.03" z="0.10">
-        <origin xyz="0 0 -0.05" rpy="0 0 0"/>
+        <origin xyz="0 0 0" rpy="0 0 0"/>
       </xacro:inertial_box>
     </link>
@@ -54,19 +72,19 @@
       <parent link="${prefix}_hip_link"/>
       <child link="${prefix}_thigh_link"/>
-      <origin xyz="${thigh_xyz}" rpy="0 0 0"/>
+      <origin xyz="${thigh_xyz}" rpy="0 ${thigh_rpy} 0"/>
       <axis xyz="0 1 0"/>
-      <limit lower="-1.571" upper="1.571" effort="2.0" velocity="5.0"/>
+      <limit lower="-2.5" upper="2.5" effort="2.0" velocity="5.0"/>
       <dynamics damping="0.05" friction="0.0"/>
     </joint>
     <link name="${prefix}_shank_link">
       <visual>
-        <origin xyz="0 0 0" rpy="0 0 0"/>
+        <origin xyz="0 0 0" rpy="0 ${mesh_shank_rpy} 0"/>
         <geometry>
-          <mesh filename="file://$(find dog_robot_description)/meshes/visual/${prefix}_shank_link.stl"/>
+          <mesh filename="package://dog_robot_description/meshes/visual/${prefix}_shank_link.stl"/>
         </geometry>
         <material name="grey"/>
       </visual>
       <collision>
-        <origin xyz="0 0 -0.0575" rpy="0 0 0"/>
+        <origin xyz="0 0 0" rpy="0 0 0"/>
         <geometry>
           <box size="0.015 0.015 0.10"/>
@@ -74,5 +92,5 @@
       </collision>
       <xacro:inertial_box mass="0.08" x="0.02" y="0.02" z="0.115">
-        <origin xyz="0 0 -0.0575" rpy="0 0 0"/>
+        <origin xyz="0 0 0" rpy="0 0 0"/>
       </xacro:inertial_box>
     </link>
@@ -80,20 +98,21 @@
       <parent link="${prefix}_thigh_link"/>
       <child link="${prefix}_shank_link"/>
-      <origin xyz="${knee_xyz}" rpy="0 0 0"/>
+      <origin xyz="${knee_xyz}" rpy="0 ${knee_rpy} 0"/>
       <axis xyz="0 1 0"/>
-      <limit lower="0.0" upper="2.617" effort="2.0" velocity="5.0"/>
+      <limit lower="-2.5" upper="2.5" effort="2.0" velocity="5.0"/>
       <dynamics damping="0.05" friction="0.0"/>
     </joint>
     <link name="${prefix}_foot_link">
       <visual>
-        <origin xyz="0 0 0" rpy="0 0 0"/>
+        <origin xyz="0 0 0" rpy="0 ${mesh_foot_rpy} 0"/>
         <geometry>
-          <mesh filename="file://$(find dog_robot_description)/meshes/visual/${prefix}_foot_link.stl"/>
+          <mesh filename="package://dog_robot_description/meshes/visual/${prefix}_foot_link.stl"/>
         </geometry>
         <material name="dark_grey"/>
       </visual>
-      <!-- Sphere collision (mesh foot caused ODE contact instability). -->
+      <!-- Sphere collision (mesh foot caused ODE contact instability).
+           foot_sphere_xyz is expressed in the rotated foot_link frame. -->
       <collision>
-        <origin xyz="0.042 0 -0.029" rpy="0 0 0"/>
+        <origin xyz="${foot_sphere_xyz}" rpy="0 0 0"/>
         <geometry>
           <sphere radius="0.018"/>

Commit message: refactor(urdf): per-leg DH config + mesh compensation in dog_robot.urdf.xacro
Co-Authored-By: Claude Sonnet 4.6 <noreply@anthropic.com>

File: dog_robot_ws/src/dog_robot_description/urdf/dog_robot.urdf.xacro (robot description, xacro)
@@ -24,55 +24,46 @@
     </xacro:inertial_box>
   </link>
-  <!-- Joint origins measured from CAD (scripts/compute_joints.py).
-       The thigh/knee rpy_y values and compensating mesh rpy_y values
-       rotate the thigh and shank link frames so knee_xyz and foot_xyz
-       lie along -Z. This makes CHAMP's IK trivially produce ~0 for
-       thigh_pitch/knee_pitch when the foot is directly below the hip.
-       foot_sphere_xyz is the original (0.042, 0, -0.029) collision
-       sphere offset re-expressed in the rotated foot_link frame:
-       sphere_new = Ry(-(thigh_rpy + knee_rpy)) * sphere_old. -->
+  <!-- Modified DH (Craig) configuration. One symmetric DH table for all 4 legs;
+       per-leg variation lives entirely in the base_to_hip_* and mesh_* params.
+       L_hh/L_th/L_sh computed from CAD by scripts/compute_dh_lengths.py;
+       mesh xyz/rpy computed by scripts/compute_visual_compensation.py. -->
+  <xacro:property name="L_hh" value="0.02553"/>
+  <xacro:property name="L_th" value="0.11725"/>
+  <xacro:property name="L_sh" value="0.07043"/>
   <xacro:leg prefix="FL"
-             hip_xyz="0.07480 0.04000 0.03510"
-             thigh_xyz="0.02520 0.02536 -0.01317"
-             knee_xyz="0.0 0.04102 -0.10984"
-             foot_xyz="0.0 -0.01922 -0.06773"
-             thigh_rpy="0.94261"
-             knee_rpy="-1.93175"
-             mesh_thigh_rpy="-0.94261"
-             mesh_shank_rpy="0.98914"
-             mesh_foot_rpy="0.98914"
-             foot_sphere_xyz="0 0 -0.050"/>
+             base_to_hip_xyz="0.07480 0.04000 0.03510"
+             base_to_hip_rpy="0 1.5707963 0"
+             L_hh="${L_hh}" L_th="${L_th}" L_sh="${L_sh}"
+             mesh_hip_xyz="0.0 0.0 0.0" mesh_hip_rpy="0.00000 -1.57080 0.00000"
+             mesh_thigh_xyz="-0.00033 0.01317 0.02536" mesh_thigh_rpy="1.57080 0.00000 0.94261"
+             mesh_shank_xyz="-0.11725 0.04102 -0.10984" mesh_shank_rpy="3.14159 -1.20984 3.14159"
+             mesh_foot_xyz="-0.07043 -0.01922 -0.06773" mesh_foot_rpy="0.00000 0.00000 0.00000"
+             foot_sphere_xyz="0 0 0"/>
   <xacro:leg prefix="FR"
-             hip_xyz="0.07480 -0.04000 0.03510"
-             thigh_xyz="0.02520 -0.02570 -0.01250"
-             knee_xyz="0.0 -0.04270 -0.10920"
-             foot_xyz="0.0 0.01826 -0.06802"
-             thigh_rpy="0.93698"
-             knee_rpy="-1.91411"
-             mesh_thigh_rpy="-0.93698"
-             mesh_shank_rpy="0.97713"
-             mesh_foot_rpy="0.97713"
-             foot_sphere_xyz="0 0 -0.050"/>
+             base_to_hip_xyz="0.07480 -0.04000 0.03510"
+             base_to_hip_rpy="0 1.5707963 3.1415927"
+             L_hh="${L_hh}" L_th="${L_th}" L_sh="${L_sh}"
+             mesh_hip_xyz="0.0 0.0 0.0" mesh_hip_rpy="0.00000 1.57080 -3.14159"
+             mesh_thigh_xyz="-0.00033 0.0125 -0.0257" mesh_thigh_rpy="1.57080 0.00000 0.93698"
+             mesh_shank_xyz="-0.11725 -0.0427 -0.1092" mesh_shank_rpy="3.14159 -1.22748 3.14159"
+             mesh_foot_xyz="-0.07043 0.01826 -0.06802" mesh_foot_rpy="0.00000 0.00000 0.00000"
+             foot_sphere_xyz="0 0 0"/>
   <xacro:leg prefix="BL"
-             hip_xyz="-0.07480 0.04000 0.03510"
-             thigh_xyz="-0.02520 0.02536 -0.01318"
-             knee_xyz="0.0 0.04082 -0.10992"
-             foot_xyz="0.0 -0.01906 -0.06742"
-             thigh_rpy="0.86151"
-             knee_rpy="-1.96488"
-             mesh_thigh_rpy="-0.86151"
-             mesh_shank_rpy="1.10337"
-             mesh_foot_rpy="1.10337"
-             foot_sphere_xyz="0 0 -0.050"/>
+             base_to_hip_xyz="-0.07480 0.04000 0.03510"
+             base_to_hip_rpy="0 1.5707963 0"
+             L_hh="${L_hh}" L_th="${L_th}" L_sh="${L_sh}"
+             mesh_hip_xyz="0.0 0.0 0.0" mesh_hip_rpy="0.00000 -1.57080 0.00000"
+             mesh_thigh_xyz="-0.05073 0.01318 0.02536" mesh_thigh_rpy="1.57080 0.00000 0.86151"
+             mesh_shank_xyz="-0.11725 0.04082 -0.10992" mesh_shank_rpy="3.14159 -1.17671 3.14159"
+             mesh_foot_xyz="-0.07043 -0.01906 -0.06742" mesh_foot_rpy="0.00000 0.00000 0.00000"
+             foot_sphere_xyz="0 0 0"/>
   <xacro:leg prefix="BR"
-             hip_xyz="-0.07480 -0.04000 0.03510"
-             thigh_xyz="-0.02520 -0.02570 -0.01250"
-             knee_xyz="0.0 -0.04270 -0.10920"
-             foot_xyz="0.0 0.01842 -0.06838"
-             thigh_rpy="0.86324"
-             knee_rpy="-1.95214"
-             mesh_thigh_rpy="-0.86324"
-             mesh_shank_rpy="1.08890"
-             mesh_foot_rpy="1.08890"
-             foot_sphere_xyz="0 0 -0.050"/>
+             base_to_hip_xyz="-0.07480 -0.04000 0.03510"
+             base_to_hip_rpy="0 1.5707963 3.1415927"
+             L_hh="${L_hh}" L_th="${L_th}" L_sh="${L_sh}"
+             mesh_hip_xyz="0.0 0.0 0.0" mesh_hip_rpy="0.00000 1.57080 -3.14159"
+             mesh_thigh_xyz="-0.05073 0.0125 -0.0257" mesh_thigh_rpy="1.57080 0.00000 0.86324"
+             mesh_shank_xyz="-0.11725 -0.0427 -0.1092" mesh_shank_rpy="3.14159 -1.18945 3.14159"
+             mesh_foot_xyz="-0.07043 0.01842 -0.06838" mesh_foot_rpy="0.00000 0.00000 0.00000"
+             foot_sphere_xyz="0 0 0"/>
 </robot>

Commit message: feat(urdf): wire derived DH params (d_thigh, d_knee) into all 4 legs
Replace old L_hh/L_th/L_sh property block with full set of derived MDH
values (mean across 4 legs from scripts/derive_dh_frames.py): L_hh,
L_th, L_sh, d_thigh, d_knee, d_foot, alpha_thigh. Forward all seven
params explicitly through every leg invocation (FL, FR, BL, BR);
base_to_hip_xyz/rpy untouched.

Co-Authored-By: Claude Sonnet 4.6 <noreply@anthropic.com>

File: dog_robot_ws/src/dog_robot_description/urdf/dog_robot.urdf.xacro (robot description, xacro)
@@ -30,11 +30,18 @@
        scripts/bake_meshes_to_link_frame.py); URDF visual <origin> is
        identity for every link. -->
-  <xacro:property name="L_hh" value="0.02553"/>
-  <xacro:property name="L_th" value="0.11725"/>
-  <xacro:property name="L_sh" value="0.07043"/>
+  <!-- Generated DH params (mean across 4 legs) — see scripts/derive_dh_frames.py -->
+  <xacro:property name="L_hh"        value="0.012836"/>
+  <xacro:property name="L_th"        value="0.109541"/>
+  <xacro:property name="L_sh"        value="0.070430"/>
+  <xacro:property name="d_thigh"     value="0.025531"/>
+  <xacro:property name="d_knee"      value="0.041810"/>
+  <xacro:property name="d_foot"      value="0.000000"/>
+  <xacro:property name="alpha_thigh" value="-1.5707963"/>
   <xacro:leg prefix="FL"
              base_to_hip_xyz="0.07480 0.04000 0.03510"
              base_to_hip_rpy="0 1.5707963 0"
              L_hh="${L_hh}" L_th="${L_th}" L_sh="${L_sh}"
+             d_thigh="${d_thigh}" d_knee="${d_knee}" d_foot="${d_foot}"
+             alpha_thigh="${alpha_thigh}"
              foot_sphere_xyz="0 0 0"/>
   <xacro:leg prefix="FR"
@@ -42,4 +49,6 @@
              base_to_hip_rpy="0 1.5707963 3.1415927"
              L_hh="${L_hh}" L_th="${L_th}" L_sh="${L_sh}"
+             d_thigh="${d_thigh}" d_knee="${d_knee}" d_foot="${d_foot}"
+             alpha_thigh="${alpha_thigh}"
              foot_sphere_xyz="0 0 0"/>
   <xacro:leg prefix="BL"
@@ -47,4 +56,6 @@
              base_to_hip_rpy="0 1.5707963 0"
              L_hh="${L_hh}" L_th="${L_th}" L_sh="${L_sh}"
+             d_thigh="${d_thigh}" d_knee="${d_knee}" d_foot="${d_foot}"
+             alpha_thigh="${alpha_thigh}"
              foot_sphere_xyz="0 0 0"/>
   <xacro:leg prefix="BR"
@@ -52,4 +63,6 @@
              base_to_hip_rpy="0 1.5707963 3.1415927"
              L_hh="${L_hh}" L_th="${L_th}" L_sh="${L_sh}"
+             d_thigh="${d_thigh}" d_knee="${d_knee}" d_foot="${d_foot}"
+             alpha_thigh="${alpha_thigh}"
              foot_sphere_xyz="0 0 0"/>
 </robot>
