Commit message: feat(urdf): per-leg exact joint origins (joint-attached frames)
leg.xacro takes full (xyz,rpy) per joint; dog_robot.urdf.xacro passes the
exact per-leg transforms from link_params/urdf_joints.yaml. Knee limit
widened to [-2.617, 0.5] for the new bent-knee sign. Adds
test_urdf_link_consistency: URDF FK == kinematics_link.fk_leg for all 4 legs.

Co-Authored-By: Claude Opus 4.7 <noreply@anthropic.com>

File: dog_robot_ws/src/dog_robot_description/urdf/dog_robot.urdf.xacro (robot description, xacro)
@@ -24,45 +24,46 @@
     </xacro:inertial_box>
   </link>
-  <!-- Modified DH (Craig) configuration. One symmetric DH table for all 4 legs;
-       per-leg variation lives entirely in the base_to_hip_* params.
-       L_hh/L_th/L_sh computed from CAD by scripts/compute_dh_lengths.py.
-       Visual meshes are pre-baked in meshes/visual_dh/ (see
-       scripts/bake_meshes_to_link_frame.py); URDF visual <origin> is
-       identity for every link. -->
-  <!-- Generated DH params (mean across 4 legs) — see scripts/derive_dh_frames.py -->
-  <xacro:property name="L_hh"        value="0.012836"/>
-  <xacro:property name="L_th"        value="0.109541"/>
-  <xacro:property name="L_sh"        value="0.070430"/>
-  <xacro:property name="d_thigh"     value="0.025531"/>
-  <xacro:property name="d_knee"      value="0.041810"/>
-  <xacro:property name="d_foot"      value="0.000000"/>
-  <xacro:property name="alpha_thigh" value="-1.5707963"/>
+  <!-- Joint-attached frame configuration (see
+       docs/superpowers/specs/2026-05-26-joint-frame-export-design.md).
+       Each joint origin is the exact (xyz, rpy) transform in the parent frame,
+       per leg (front/back legs differ; left/right mirror). Generated by
+       scripts/derive_joint_frames.py → config/{link_params,urdf_joints}.yaml.
+       Visual meshes in meshes/visual_dh/ are vertex-aligned to these frames, so
+       every URDF visual <origin> is identity. -->
   <xacro:leg prefix="FL"
-             base_to_hip_xyz="0.07480 0.04000 0.03510"
-             base_to_hip_rpy="0 1.5707963 0"
-             L_hh="${L_hh}" L_th="${L_th}" L_sh="${L_sh}"
-             d_thigh="${d_thigh}" d_knee="${d_knee}" d_foot="${d_foot}"
-             alpha_thigh="${alpha_thigh}"
-             foot_sphere_xyz="0 0 0"/>
+             base_to_hip_xyz="0.07480000 0.04000000 0.03510000"
+             base_to_hip_rpy="0.00000000 -0.00000000 0.78860214"
+             hip_to_thigh_xyz="0.03575292 0.00000000 -0.01317100"
+             hip_to_thigh_rpy="1.57079633 0.62818252 2.35299051"
+             thigh_to_knee_xyz="0.10984469 0.00000000 0.04101700"
+             thigh_to_knee_rpy="0.00000000 -0.00000000 -1.93205288"
+             knee_to_foot_xyz="0.06769627 -0.00000000 -0.01917900"
+             knee_to_foot_rpy="1.57079633 -0.00000000 -0.58135726"/>
   <xacro:leg prefix="FR"
-             base_to_hip_xyz="0.07480 -0.04000 0.03510"
-             base_to_hip_rpy="0 1.5707963 3.1415927"
-             L_hh="${L_hh}" L_th="${L_th}" L_sh="${L_sh}"
-             d_thigh="${d_thigh}" d_knee="${d_knee}" d_foot="${d_foot}"
-             alpha_thigh="${alpha_thigh}"
-             foot_sphere_xyz="0 0 0"/>
+             base_to_hip_xyz="0.07480000 -0.04000000 0.03510000"
+             base_to_hip_rpy="-0.00000000 -0.00000000 -0.79522103"
+             hip_to_thigh_xyz="0.03599347 0.00000000 -0.01250000"
+             hip_to_thigh_rpy="1.57079633 0.63382895 -2.34637162"
+             thigh_to_knee_xyz="0.10920171 0.00000000 -0.04270000"
+             thigh_to_knee_rpy="0.00000000 -0.00000000 -1.91446402"
+             knee_to_foot_xyz="0.06801469 0.00000000 0.01830000"
+             knee_to_foot_rpy="1.57079633 -0.00000000 -0.59329969"/>
   <xacro:leg prefix="BL"
-             base_to_hip_xyz="-0.07480 0.04000 0.03510"
-             base_to_hip_rpy="0 1.5707963 0"
-             L_hh="${L_hh}" L_th="${L_th}" L_sh="${L_sh}"
-             d_thigh="${d_thigh}" d_knee="${d_knee}" d_foot="${d_foot}"
-             alpha_thigh="${alpha_thigh}"
-             foot_sphere_xyz="0 0 0"/>
+             base_to_hip_xyz="-0.07480000 0.04000000 0.03510000"
+             base_to_hip_rpy="0.00000000 -0.00000000 2.35301023"
+             hip_to_thigh_xyz="0.03575221 0.00000000 -0.01317500"
+             hip_to_thigh_rpy="1.57079633 0.70925979 0.78858243"
+             thigh_to_knee_xyz="0.10991717 0.00000000 0.04082200"
+             thigh_to_knee_rpy="0.00000000 -0.00000000 -1.96558097"
+             knee_to_foot_xyz="0.06742180 0.00000000 -0.01908300"
+             knee_to_foot_rpy="1.57079633 -0.00000000 -0.46675189"/>
   <xacro:leg prefix="BR"
-             base_to_hip_xyz="-0.07480 -0.04000 0.03510"
-             base_to_hip_rpy="0 1.5707963 3.1415927"
-             L_hh="${L_hh}" L_th="${L_th}" L_sh="${L_sh}"
-             d_thigh="${d_thigh}" d_knee="${d_knee}" d_foot="${d_foot}"
-             alpha_thigh="${alpha_thigh}"
-             foot_sphere_xyz="0 0 0"/>
+             base_to_hip_xyz="-0.07480000 -0.04000000 0.03510000"
+             base_to_hip_rpy="0.00000000 -0.00000000 -2.34637162"
+             hip_to_thigh_xyz="0.03599347 0.00000000 -0.01250000"
+             hip_to_thigh_rpy="1.57079633 0.70757143 -0.79522103"
+             thigh_to_knee_xyz="0.10920166 0.00000000 -0.04270000"
+             thigh_to_knee_rpy="0.00000000 -0.00000000 -1.95171579"
+             knee_to_foot_xyz="0.06838818 0.00000000 0.01840000"
+             knee_to_foot_rpy="1.57079633 -0.00000000 -0.48230543"/>
 </robot>

File: dog_robot_ws/src/dog_robot_description/urdf/leg.xacro (robot description, xacro)
@@ -3,7 +3,7 @@
   <xacro:macro name="leg" params="prefix
                                   base_to_hip_xyz base_to_hip_rpy
-                                  L_hh L_th L_sh
-                                  d_thigh:='0' d_knee:='0' d_foot:='0'
-                                  alpha_thigh:='-1.5707963'
+                                  hip_to_thigh_xyz hip_to_thigh_rpy
+                                  thigh_to_knee_xyz thigh_to_knee_rpy
+                                  knee_to_foot_xyz knee_to_foot_rpy
                                   foot_sphere_xyz:='0 0 0'">
     <link name="${prefix}_hip_link">
@@ -50,5 +50,5 @@
       <parent link="${prefix}_hip_link"/>
       <child link="${prefix}_thigh_link"/>
-      <origin xyz="${L_hh} ${d_thigh} 0" rpy="${alpha_thigh} 0 0"/>
+      <origin xyz="${hip_to_thigh_xyz}" rpy="${hip_to_thigh_rpy}"/>
       <axis xyz="0 0 1"/>
       <limit lower="-1.571" upper="1.571" effort="10.0" velocity="8.0"/>
@@ -74,7 +74,7 @@
       <parent link="${prefix}_thigh_link"/>
       <child link="${prefix}_shank_link"/>
-      <origin xyz="${L_th} 0 ${d_knee}" rpy="0 0 0"/>
+      <origin xyz="${thigh_to_knee_xyz}" rpy="${thigh_to_knee_rpy}"/>
       <axis xyz="0 0 1"/>
-      <limit lower="0.0" upper="2.617" effort="10.0" velocity="8.0"/>
+      <limit lower="-2.617" upper="0.5" effort="10.0" velocity="8.0"/>
       <dynamics damping="0.5" friction="0.0"/>
     </joint>
@@ -98,5 +98,5 @@
       <parent link="${prefix}_shank_link"/>
       <child link="${prefix}_foot_link"/>
-      <origin xyz="${L_sh} 0 ${d_foot}" rpy="0 0 0"/>
+      <origin xyz="${knee_to_foot_xyz}" rpy="${knee_to_foot_rpy}"/>
     </joint>
   </xacro:macro>

Commit message: chore: strip Gazebo / CHAMP / controller stack down to kinematic core
Delete entire packages: champ/, dog_robot_config/, dog_robot_control/.
Delete Gazebo plumbing in dog_robot_description: gazebo.xacro,
ros2_control.xacro, inertial.xacro, launch/gazebo.launch.py,
config/ros2_controllers.yaml, config/dh_link_placements.yaml, and the
legacy DH-era scripts (compute_dh_lengths, derive_dh_frames,
compute_visual_compensation).
Delete legacy kinematics_dh.py + leg_config.py + config/dh_params.yaml;
rewire dog_robot_kinematics.__init__ to expose only kinematics_link.
Drop xacro:inertial_* calls from leg.xacro and base_link.
Trim dog_robot_description package.xml exec_depends to xacro / urdf /
RSP / RViz / joint_state_publisher; CMakeLists drops the now-empty
launch/.
test_urdf.py: use relative path (Path(__file__)…), not the hardcoded
main-workspace path.
Trim scripts/dog_kill_all.sh patterns to the kinematic-viz set.

URDF post-cleanup: 17 links, 12 revolute joints, 0 inertials.
check_urdf passes.

Co-Authored-By: Claude Opus 4.7 <noreply@anthropic.com>

File: dog_robot_ws/src/dog_robot_description/urdf/dog_robot.urdf.xacro (robot description, xacro)
@@ -2,8 +2,5 @@
 <robot xmlns:xacro="http://www.ros.org/wiki/xacro" name="dog_robot">
   <xacro:include filename="$(find dog_robot_description)/urdf/materials.xacro"/>
-  <xacro:include filename="$(find dog_robot_description)/urdf/inertial.xacro"/>
   <xacro:include filename="$(find dog_robot_description)/urdf/leg.xacro"/>
-  <xacro:include filename="$(find dog_robot_description)/urdf/gazebo.xacro"/>
-  <xacro:include filename="$(find dog_robot_description)/urdf/ros2_control.xacro"/>
   <link name="base_link">
     <visual>
@@ -20,7 +17,4 @@
       </geometry>
     </collision>
-    <xacro:inertial_box mass="0.80" x="0.200" y="0.080" z="0.060">
-      <origin xyz="0 0 0" rpy="0 0 0"/>
-    </xacro:inertial_box>
   </link>
   <!-- Joint-attached frame configuration (see

File: dog_robot_ws/src/dog_robot_description/urdf/leg.xacro (robot description, xacro)
@@ -19,7 +19,4 @@
         <geometry><box size="0.03 0.03 0.03"/></geometry>
       </collision>
-      <xacro:inertial_box mass="0.15" x="0.04" y="0.04" z="0.04">
-        <origin xyz="0 0 0" rpy="0 0 0"/>
-      </xacro:inertial_box>
     </link>
     <joint name="${prefix}_hip_yaw" type="revolute">
@@ -43,7 +40,4 @@
         <geometry><box size="0.02 0.02 0.08"/></geometry>
       </collision>
-      <xacro:inertial_box mass="0.10" x="0.03" y="0.03" z="0.10">
-        <origin xyz="0 0 0" rpy="0 0 0"/>
-      </xacro:inertial_box>
     </link>
     <joint name="${prefix}_thigh_pitch" type="revolute">
@@ -67,7 +61,4 @@
         <geometry><box size="0.015 0.015 0.10"/></geometry>
       </collision>
-      <xacro:inertial_box mass="0.08" x="0.02" y="0.02" z="0.115">
-        <origin xyz="0 0 0" rpy="0 0 0"/>
-      </xacro:inertial_box>
     </link>
     <joint name="${prefix}_knee_pitch" type="revolute">
@@ -91,7 +82,4 @@
         <geometry><sphere radius="0.018"/></geometry>
       </collision>
-      <xacro:inertial_sphere mass="0.02" radius="0.015">
-        <origin xyz="0 0 0" rpy="0 0 0"/>
-      </xacro:inertial_sphere>
     </link>
     <joint name="${prefix}_foot_fixed" type="fixed">

Commit message: fix(urdf): hip axis = body +X (REP-103 roll), rename hip_yaw -> hip_roll
The first leg joint was rotating about world Z (yaw / vertical) — a CAD
artefact from the joint-frame export that overrode the natural hip-roll /
abduction axis. ROS REP-103 + standard quadruped convention puts that
joint about body +X. Reorienting the hip link frame to Z = body +X
uniformly across all 4 legs.

derive_joint_frames.py: HIP_AXIS_URDF = [1, 0, 0]; regenerates
joint_frames.yaml, link_params.yaml, urdf_joints.yaml + matching
hard-coded values in dog_robot.urdf.xacro.

kinematics_link FK/IK math is unchanged (still Rz at every joint after
the per-link frame reorientation captured in LinkParams). Tests retuned
where the workspace shape shifted (hip roll +/-0.2 rad is a generous
operating range; the prior +/-0.4 hit edge cases that aren't physical).

Visual meshes are still baked to the old hip frame, so they will appear
tipped 90 deg in RViz until re-exported via FreeCAD MCP — TF axes and
joint behavior are correct.

76/76 tests pass (description 2/2, kinematics 23/23, kinematic_viz 51/51).

Co-Authored-By: Claude Opus 4.7 <noreply@anthropic.com>

File: dog_robot_ws/src/dog_robot_description/urdf/dog_robot.urdf.xacro (robot description, xacro)
@@ -27,7 +27,7 @@
   <xacro:leg prefix="FL"
              base_to_hip_xyz="0.07480000 0.04000000 0.03510000"
-             base_to_hip_rpy="0.00000000 -0.00000000 0.78860214"
-             hip_to_thigh_xyz="0.03575292 0.00000000 -0.01317100"
-             hip_to_thigh_rpy="1.57079633 0.62818252 2.35299051"
+             base_to_hip_rpy="1.57079633 0.47898407 1.57079633"
+             hip_to_thigh_xyz="0.02857807 0.00000000 0.02520000"
+             hip_to_thigh_rpy="-1.57079633 0.94261381 -1.09181226"
              thigh_to_knee_xyz="0.10984469 0.00000000 0.04101700"
              thigh_to_knee_rpy="0.00000000 -0.00000000 -1.93205288"
@@ -36,7 +36,7 @@
   <xacro:leg prefix="FR"
              base_to_hip_xyz="0.07480000 -0.04000000 0.03510000"
-             base_to_hip_rpy="-0.00000000 -0.00000000 -0.79522103"
-             hip_to_thigh_xyz="0.03599347 0.00000000 -0.01250000"
-             hip_to_thigh_rpy="1.57079633 0.63382895 -2.34637162"
+             base_to_hip_rpy="-1.57079633 0.45269343 -1.57079633"
+             hip_to_thigh_xyz="0.02857866 0.00000000 0.02520000"
+             hip_to_thigh_rpy="-1.57079633 0.93696738 1.11810290"
              thigh_to_knee_xyz="0.10920171 0.00000000 -0.04270000"
              thigh_to_knee_rpy="0.00000000 -0.00000000 -1.91446402"
@@ -45,7 +45,7 @@
   <xacro:leg prefix="BL"
              base_to_hip_xyz="-0.07480000 0.04000000 0.03510000"
-             base_to_hip_rpy="0.00000000 -0.00000000 2.35301023"
-             hip_to_thigh_xyz="0.03575221 0.00000000 -0.01317500"
-             hip_to_thigh_rpy="1.57079633 0.70925979 0.78858243"
+             base_to_hip_rpy="1.57079633 0.47912441 1.57079633"
+             hip_to_thigh_xyz="0.02857903 -0.00000000 -0.02520000"
+             hip_to_thigh_rpy="-1.57079633 0.86153654 -1.09167192"
              thigh_to_knee_xyz="0.10991717 0.00000000 0.04082200"
              thigh_to_knee_rpy="0.00000000 -0.00000000 -1.96558097"
@@ -54,7 +54,7 @@
   <xacro:leg prefix="BR"
              base_to_hip_xyz="-0.07480000 -0.04000000 0.03510000"
-             base_to_hip_rpy="0.00000000 -0.00000000 -2.34637162"
-             hip_to_thigh_xyz="0.03599347 0.00000000 -0.01250000"
-             hip_to_thigh_rpy="1.57079633 0.70757143 -0.79522103"
+             base_to_hip_rpy="-1.57079633 0.45269343 -1.57079633"
+             hip_to_thigh_xyz="0.02857866 0.00000000 -0.02520000"
+             hip_to_thigh_rpy="-1.57079633 0.86322489 1.11810290"
              thigh_to_knee_xyz="0.10920166 0.00000000 -0.04270000"
              thigh_to_knee_rpy="0.00000000 -0.00000000 -1.95171579"

File: dog_robot_ws/src/dog_robot_description/urdf/leg.xacro (robot description, xacro)
@@ -20,5 +20,5 @@
       </collision>
     </link>
-    <joint name="${prefix}_hip_yaw" type="revolute">
+    <joint name="${prefix}_hip_roll" type="revolute">
       <parent link="base_link"/>
       <child link="${prefix}_hip_link"/>
