Commit message: tune(champ): align gait + ros_control + URDF effort with CHAMP defaults
Big walking quality improvement:
- gait: nominal_height 0.16 → 0.20, odom_scaler 1.0 → 0.9,
  max_linear_velocity_x 0.3 → 0.5 (match CHAMP defaults)
- ros_control gains: p 20 → 80, i 0.05 → 0.15, d 0.2 → 0.8,
  i_clamp 0.5 → 2.0 (was 5x too low, joints sluggish)
- URDF revolute joint effort 2.0 → 5.0 N·m, velocity 5.0 → 8.0 rad/s
  (allow PID output to reach actuators without URDF-level clamp)

Verified in Gazebo:
- Idle drift dropped from 36 mm/s to ~0 mm/s (robot holds stance)
- Forward cmd_vel.x=0.1 → robot moves +16 mm/s in correct +x direction
- Robot upright throughout (w=0.999)

Speed tracking still lower than commanded (~16% of target) but
direction and gait pattern now physically correct.

Co-Authored-By: Claude Opus 4.7 (1M context) <noreply@anthropic.com>

File: dog_robot_ws/src/dog_robot_description/urdf/leg.xacro (robot description, xacro)
@@ -48,5 +48,5 @@
       <origin xyz="${hip_xyz}" rpy="0 0 0"/>
       <axis xyz="1 0 0"/>
-      <limit lower="-0.785" upper="0.785" effort="2.0" velocity="5.0"/>
+      <limit lower="-0.785" upper="0.785" effort="5.0" velocity="8.0"/>
       <dynamics damping="0.05" friction="0.0"/>
     </joint>
@@ -74,5 +74,5 @@
       <origin xyz="${thigh_xyz}" rpy="0 ${thigh_rpy} 0"/>
       <axis xyz="0 1 0"/>
-      <limit lower="-2.5" upper="2.5" effort="2.0" velocity="5.0"/>
+      <limit lower="-2.5" upper="2.5" effort="5.0" velocity="8.0"/>
       <dynamics damping="0.05" friction="0.0"/>
     </joint>
@@ -100,5 +100,5 @@
       <origin xyz="${knee_xyz}" rpy="0 ${knee_rpy} 0"/>
       <axis xyz="0 1 0"/>
-      <limit lower="-2.5" upper="2.5" effort="2.0" velocity="5.0"/>
+      <limit lower="-2.5" upper="2.5" effort="5.0" velocity="8.0"/>
       <dynamics damping="0.05" friction="0.0"/>
     </joint>

Commit message: refactor(urdf): DH-aligned joint origins in leg.xacro macro
Co-Authored-By: Claude Sonnet 4.6 <noreply@anthropic.com>

File: dog_robot_ws/src/dog_robot_description/urdf/leg.xacro (robot description, xacro)
@@ -1,28 +1,15 @@
 <?xml version="1.0"?>
 <robot xmlns:xacro="http://www.ros.org/wiki/xacro" name="dog_robot_leg">
-  <!--
-    Joint origins are measured from CAD (see scripts/compute_joints.py).
-    CHAMP-IK-compatible surgery:
-      - thigh_pitch joint frame is rotated by Ry(thigh_rpy) so the
-        knee_xyz lies along -Z (kills ik_alpha bias term).
-      - knee_pitch joint frame is rotated by Ry(knee_rpy) so the
-        foot_xyz lies along -Z (kills ik_beta bias term).
-      - Visual meshes get compensating Ry rotations so the rendered
-        geometry still matches the original CAD pose.
-      - Collision boxes on thigh/shank are reset to xyz=0 rpy=0; the
-        original z-offset was tuned for the un-rotated frame and is
-        not worth re-deriving (boxes are small and approximately
-        symmetric about link origin).
-      - Foot collision sphere xyz must be passed in already expressed
-        in the rotated foot_link frame.
-  -->
   <xacro:macro name="leg" params="prefix
-                                  hip_xyz thigh_xyz knee_xyz foot_xyz
-                                  thigh_rpy:=0 knee_rpy:=0
-                                  mesh_thigh_rpy:=0 mesh_shank_rpy:=0 mesh_foot_rpy:=0
-                                  foot_sphere_xyz:='0.042 0 -0.029'">
+                                  base_to_hip_xyz base_to_hip_rpy
+                                  L_hh L_th L_sh
+                                  mesh_hip_xyz mesh_hip_rpy
+                                  mesh_thigh_xyz mesh_thigh_rpy
+                                  mesh_shank_xyz mesh_shank_rpy
+                                  mesh_foot_xyz mesh_foot_rpy
+                                  foot_sphere_xyz:='0 0 0'">
     <link name="${prefix}_hip_link">
       <visual>
-        <origin xyz="0 0 0" rpy="0 0 0"/>
+        <origin xyz="${mesh_hip_xyz}" rpy="${mesh_hip_rpy}"/>
         <geometry>
           <mesh filename="package://dog_robot_description/meshes/visual/${prefix}_hip_link.stl"/>
@@ -30,12 +17,7 @@
         <material name="grey"/>
       </visual>
-      <!-- Small box collision keeps ODE physics active on this branch.
-           Self-collisions are disabled in gazebo.xacro so legs don't
-           prop the body up. -->
       <collision>
         <origin xyz="0 0 0" rpy="0 0 0"/>
-        <geometry>
-          <box size="0.03 0.03 0.03"/>
-        </geometry>
+        <geometry><box size="0.03 0.03 0.03"/></geometry>
       </collision>
       <xacro:inertial_box mass="0.15" x="0.04" y="0.04" z="0.04">
@@ -46,6 +28,6 @@
       <parent link="base_link"/>
       <child link="${prefix}_hip_link"/>
-      <origin xyz="${hip_xyz}" rpy="0 0 0"/>
-      <axis xyz="1 0 0"/>
+      <origin xyz="${base_to_hip_xyz}" rpy="${base_to_hip_rpy}"/>
+      <axis xyz="0 0 1"/>
       <limit lower="-0.785" upper="0.785" effort="5.0" velocity="8.0"/>
       <dynamics damping="0.05" friction="0.0"/>
@@ -53,5 +35,5 @@
     <link name="${prefix}_thigh_link">
       <visual>
-        <origin xyz="0 0 0" rpy="0 ${mesh_thigh_rpy} 0"/>
+        <origin xyz="${mesh_thigh_xyz}" rpy="${mesh_thigh_rpy}"/>
         <geometry>
           <mesh filename="package://dog_robot_description/meshes/visual/${prefix}_thigh_link.stl"/>
@@ -61,7 +43,5 @@
       <collision>
         <origin xyz="0 0 0" rpy="0 0 0"/>
-        <geometry>
-          <box size="0.02 0.02 0.08"/>
-        </geometry>
+        <geometry><box size="0.02 0.02 0.08"/></geometry>
       </collision>
       <xacro:inertial_box mass="0.10" x="0.03" y="0.03" z="0.10">
@@ -72,12 +52,12 @@
       <parent link="${prefix}_hip_link"/>
       <child link="${prefix}_thigh_link"/>
-      <origin xyz="${thigh_xyz}" rpy="0 ${thigh_rpy} 0"/>
-      <axis xyz="0 1 0"/>
-      <limit lower="-2.5" upper="2.5" effort="5.0" velocity="8.0"/>
+      <origin xyz="${L_hh} 0 0" rpy="-1.5707963 0 0"/>
+      <axis xyz="0 0 1"/>
+      <limit lower="-1.571" upper="1.571" effort="5.0" velocity="8.0"/>
       <dynamics damping="0.05" friction="0.0"/>
     </joint>
     <link name="${prefix}_shank_link">
       <visual>
-        <origin xyz="0 0 0" rpy="0 ${mesh_shank_rpy} 0"/>
+        <origin xyz="${mesh_shank_xyz}" rpy="${mesh_shank_rpy}"/>
         <geometry>
           <mesh filename="package://dog_robot_description/meshes/visual/${prefix}_shank_link.stl"/>
@@ -87,7 +67,5 @@
       <collision>
         <origin xyz="0 0 0" rpy="0 0 0"/>
-        <geometry>
-          <box size="0.015 0.015 0.10"/>
-        </geometry>
+        <geometry><box size="0.015 0.015 0.10"/></geometry>
       </collision>
       <xacro:inertial_box mass="0.08" x="0.02" y="0.02" z="0.115">
@@ -98,12 +76,12 @@
       <parent link="${prefix}_thigh_link"/>
       <child link="${prefix}_shank_link"/>
-      <origin xyz="${knee_xyz}" rpy="0 ${knee_rpy} 0"/>
-      <axis xyz="0 1 0"/>
-      <limit lower="-2.5" upper="2.5" effort="5.0" velocity="8.0"/>
+      <origin xyz="${L_th} 0 0" rpy="0 0 0"/>
+      <axis xyz="0 0 1"/>
+      <limit lower="0.0" upper="2.617" effort="5.0" velocity="8.0"/>
       <dynamics damping="0.05" friction="0.0"/>
     </joint>
     <link name="${prefix}_foot_link">
       <visual>
-        <origin xyz="0 0 0" rpy="0 ${mesh_foot_rpy} 0"/>
+        <origin xyz="${mesh_foot_xyz}" rpy="${mesh_foot_rpy}"/>
         <geometry>
           <mesh filename="package://dog_robot_description/meshes/visual/${prefix}_foot_link.stl"/>
@@ -111,11 +89,7 @@
         <material name="dark_grey"/>
       </visual>
-      <!-- Sphere collision (mesh foot caused ODE contact instability).
-           foot_sphere_xyz is expressed in the rotated foot_link frame. -->
       <collision>
         <origin xyz="${foot_sphere_xyz}" rpy="0 0 0"/>
-        <geometry>
-          <sphere radius="0.018"/>
-        </geometry>
+        <geometry><sphere radius="0.018"/></geometry>
       </collision>
       <xacro:inertial_sphere mass="0.02" radius="0.015">
@@ -126,5 +100,5 @@
       <parent link="${prefix}_shank_link"/>
       <child link="${prefix}_foot_link"/>
-      <origin xyz="${foot_xyz}" rpy="0 0 0"/>
+      <origin xyz="${L_sh} 0 0" rpy="0 0 0"/>
     </joint>
   </xacro:macro>

Commit message: feat(urdf): leg.xacro accepts d_thigh/d_knee/d_foot/alpha_thigh
Add optional DH offset params (d_thigh, d_knee, d_foot, alpha_thigh)
to the leg macro with safe defaults (0 / -1.5707963) so existing call
sites continue to work unchanged. Joint origins for thigh_pitch,
knee_pitch, and foot_fixed updated to use the new params.

Co-Authored-By: Claude Sonnet 4.6 <noreply@anthropic.com>

File: dog_robot_ws/src/dog_robot_description/urdf/leg.xacro (robot description, xacro)
@@ -4,4 +4,6 @@
                                   base_to_hip_xyz base_to_hip_rpy
                                   L_hh L_th L_sh
+                                  d_thigh:='0' d_knee:='0' d_foot:='0'
+                                  alpha_thigh:='-1.5707963'
                                   foot_sphere_xyz:='0 0 0'">
     <link name="${prefix}_hip_link">
@@ -48,5 +50,5 @@
       <parent link="${prefix}_hip_link"/>
       <child link="${prefix}_thigh_link"/>
-      <origin xyz="${L_hh} 0 0" rpy="-1.5707963 0 0"/>
+      <origin xyz="${L_hh} 0 ${d_thigh}" rpy="${alpha_thigh} 0 0"/>
       <axis xyz="0 0 1"/>
       <limit lower="-1.571" upper="1.571" effort="10.0" velocity="8.0"/>
@@ -72,5 +74,5 @@
       <parent link="${prefix}_thigh_link"/>
       <child link="${prefix}_shank_link"/>
-      <origin xyz="${L_th} 0 0" rpy="0 0 0"/>
+      <origin xyz="${L_th} 0 ${d_knee}" rpy="0 0 0"/>
       <axis xyz="0 0 1"/>
       <limit lower="0.0" upper="2.617" effort="10.0" velocity="8.0"/>
@@ -96,5 +98,5 @@
       <parent link="${prefix}_shank_link"/>
       <child link="${prefix}_foot_link"/>
-      <origin xyz="${L_sh} 0 0" rpy="0 0 0"/>
+      <origin xyz="${L_sh} 0 ${d_foot}" rpy="0 0 0"/>
     </joint>
   </xacro:macro>

Commit message: test(urdf-dh): consistency check with d_* offsets; fix thigh origin axis
- dh_params.yaml: update to derived values (L_hh=0.012836, L_th=0.109541,
  L_sh=0.070430) and add d_thigh=0.025531, d_knee=0.041810, d_foot=0.000000
- test_urdf_dh_consistency.py: load DHParams from yaml via _load_dh_from_yaml()
  instead of hardcoded stale values; adds yaml + pathlib imports
- leg.xacro: fix thigh_pitch origin from xyz="${L_hh} 0 ${d_thigh}" to
  xyz="${L_hh} ${d_thigh} 0" — MDH d_2 offsets along Z_2 which after
  Rx(-pi/2) lands in Y of the hip frame, not Z; previous placement was wrong
  and caused URDF FK to diverge from kinematics_dh.fk_leg

All 21 kinematics tests pass (21 passed, 0 failed).

Co-Authored-By: Claude Sonnet 4.6 <noreply@anthropic.com>

File: dog_robot_ws/src/dog_robot_description/urdf/leg.xacro (robot description, xacro)
@@ -50,5 +50,5 @@
       <parent link="${prefix}_hip_link"/>
       <child link="${prefix}_thigh_link"/>
-      <origin xyz="${L_hh} 0 ${d_thigh}" rpy="${alpha_thigh} 0 0"/>
+      <origin xyz="${L_hh} ${d_thigh} 0" rpy="${alpha_thigh} 0 0"/>
       <axis xyz="0 0 1"/>
       <limit lower="-1.571" upper="1.571" effort="10.0" velocity="8.0"/>
