Commit message: docs(readme): refresh kinematics + spawn-pose sections
- Replace DH-table description with the joint-attached link-frame model
  (per-leg fixed transforms read from link_params.yaml; fk_leg / ik_leg
  via kinematics_link).
- Document the ros2_control initial_value stand pose and the z=0.16
  spawn height that pairs with it (the 18 mm contact impulse story).
- Note the kinematic.rviz move from dog_robot_control/rviz to
  dog_robot_kinematic_viz/rviz (matches the launch files).
- Bundle the matching launch + URDF + setup.py edits.

Co-Authored-By: Claude Opus 4.7 <noreply@anthropic.com>

File: dog_robot_ws/src/dog_robot_description/urdf/ros2_control.xacro (robot description, xacro)
@@ -1,5 +1,9 @@
 <?xml version="1.0"?>
 <robot xmlns:xacro="http://www.ros.org/wiki/xacro" name="dog_robot_ros2_control">
-  <xacro:macro name="joint_iface" params="name lower upper">
+  <!-- initial_value sets the joint state at plugin Load() BEFORE physics ticks.
+       Using stand pose (thigh=-0.4146, knee=1.1498 for body_z=0.15) so feet
+       are at ground level on spawn; commanding straight legs (theta=0)
+       puts foot 18mm BELOW ground => 360 N contact impulse => explosion. -->
+  <xacro:macro name="joint_iface" params="name lower upper initial">
     <joint name="${name}">
       <command_interface name="position">
@@ -8,5 +12,7 @@
       </command_interface>
       <command_interface name="effort"/>
-      <state_interface name="position"/>
+      <state_interface name="position">
+        <param name="initial_value">${initial}</param>
+      </state_interface>
       <state_interface name="velocity"/>
     </joint>
@@ -16,16 +22,16 @@
       <plugin>gazebo_ros2_control/GazeboSystem</plugin>
     </hardware>
-    <xacro:joint_iface name="FL_hip_yaw"     lower="-0.785" upper="0.785"/>
-    <xacro:joint_iface name="FL_thigh_pitch" lower="-1.571" upper="1.571"/>
-    <xacro:joint_iface name="FL_knee_pitch"  lower="0.0"    upper="2.617"/>
-    <xacro:joint_iface name="FR_hip_yaw"     lower="-0.785" upper="0.785"/>
-    <xacro:joint_iface name="FR_thigh_pitch" lower="-1.571" upper="1.571"/>
-    <xacro:joint_iface name="FR_knee_pitch"  lower="0.0"    upper="2.617"/>
-    <xacro:joint_iface name="BL_hip_yaw"     lower="-0.785" upper="0.785"/>
-    <xacro:joint_iface name="BL_thigh_pitch" lower="-1.571" upper="1.571"/>
-    <xacro:joint_iface name="BL_knee_pitch"  lower="0.0"    upper="2.617"/>
-    <xacro:joint_iface name="BR_hip_yaw"     lower="-0.785" upper="0.785"/>
-    <xacro:joint_iface name="BR_thigh_pitch" lower="-1.571" upper="1.571"/>
-    <xacro:joint_iface name="BR_knee_pitch"  lower="0.0"    upper="2.617"/>
+    <xacro:joint_iface name="FL_hip_yaw"     lower="-0.785" upper="0.785" initial="0.0"/>
+    <xacro:joint_iface name="FL_thigh_pitch" lower="-1.571" upper="1.571" initial="-0.4146"/>
+    <xacro:joint_iface name="FL_knee_pitch"  lower="0.0"    upper="2.617" initial="1.1498"/>
+    <xacro:joint_iface name="FR_hip_yaw"     lower="-0.785" upper="0.785" initial="0.0"/>
+    <xacro:joint_iface name="FR_thigh_pitch" lower="-1.571" upper="1.571" initial="-0.4146"/>
+    <xacro:joint_iface name="FR_knee_pitch"  lower="0.0"    upper="2.617" initial="1.1498"/>
+    <xacro:joint_iface name="BL_hip_yaw"     lower="-0.785" upper="0.785" initial="0.0"/>
+    <xacro:joint_iface name="BL_thigh_pitch" lower="-1.571" upper="1.571" initial="-0.4146"/>
+    <xacro:joint_iface name="BL_knee_pitch"  lower="0.0"    upper="2.617" initial="1.1498"/>
+    <xacro:joint_iface name="BR_hip_yaw"     lower="-0.785" upper="0.785" initial="0.0"/>
+    <xacro:joint_iface name="BR_thigh_pitch" lower="-1.571" upper="1.571" initial="-0.4146"/>
+    <xacro:joint_iface name="BR_knee_pitch"  lower="0.0"    upper="2.617" initial="1.1498"/>
   </ros2_control>
 </robot>
